File: pcb/kicad/lemon-piano.kicad_sch (KiCad schematic)
At the start: 42 parts, among them J1 5V_IN, J2 LEMON_KEYS, SW1 SENS+, SW2 SENS-, U1 Nano_socket_A, U2 Nano_socket_B

Commit message: fix(pcb): v0.2.0 — real Nano orientation (erratum ADR-015) + full render suite
The photo-overlay verification caught v0.1.0's socket maps being
180°-rotated (TX1/VIN are at the ICSP end on real Nanos, D12/D13 at the
mini-USB end — verified on the official 2008 V2.2 board photo and
clones). v0.1.0 only worked inserted USB-east, where the buzzer blocks
the plug; its release folder is renamed v0.1.0-ERRATUM-do-not-fab.

v0.2.0 keeps the mechanics (USB corridor west) and fixes the maps:
keys header SOUTH (1..7 G under A0-A6), LED bar NORTH ascending
east→west, pull-ups with their pins; ground truth, schematic, netlist
and every gate re-derived — DRC 0/0/0, ERC 0/0, verify_placement/
holes/geometry PASS, fab zip under pcb/releases/v0.2.0/.

Render suite via the pcb-designer service v0.3.0 (3D models installed):
bare / dim / realistic / realistic-dim per side + photo overlay with a
real Nano image (Wikimedia Commons File:Arduino Nano.jpg, CC BY 2.0,
provenance in pcb/overlays/modules.yaml). post_route self-healing
upgrades (connectivity-based island bridging, split-net repair, exact
clearance geometry, IsOnLayer fix) in ADR-018.

Co-Authored-By: Claude Fable 5 <noreply@anthropic.com>
Connections:
- net +5V: now also U1.12 (Pin_12); no longer U2.12 (Pin_12)
- net BUZZER: now also U1.1 (Pin_1); no longer U2.1 (Pin_1)
- net GND: now also J2.8 (Pin_8), U1.14 (Pin_14), U2.4 (Pin_4); no longer J2.1 (Pin_1), U1.4 (Pin_4), U2.14 (Pin_14)
- net KEY1: now also J2.1 (Pin_1), U1.4 (Pin_4); no longer J2.8 (Pin_8), U2.4 (Pin_4)
- net KEY2: now also J2.2 (Pin_2), U1.5 (Pin_5); no longer J2.7 (Pin_7), U2.5 (Pin_5)
- net KEY3: now also J2.3 (Pin_3), U1.6 (Pin_6); no longer J2.6 (Pin_6), U2.6 (Pin_6)
- net KEY4: now also J2.4 (Pin_4), U1.7 (Pin_7); no longer J2.5 (Pin_5), U2.7 (Pin_7)
- net KEY5: now also J2.5 (Pin_5), U1.8 (Pin_8); no longer J2.4 (Pin_4), U2.8 (Pin_8)
- net KEY6: now also J2.6 (Pin_6), U1.9 (Pin_9); no longer J2.3 (Pin_3), U2.9 (Pin_9)
- net KEY7: now also J2.7 (Pin_7), U1.10 (Pin_10); no longer J2.2 (Pin_2), U2.10 (Pin_10)
- net LED1: now also U2.5 (Pin_5); no longer U1.5 (Pin_5)
- net LED10: now also U2.14 (Pin_14); no longer U1.14 (Pin_14)
- net LED2: now also U2.6 (Pin_6); no longer U1.6 (Pin_6)
- net LED3: now also U2.7 (Pin_7); no longer U1.7 (Pin_7)
- net LED4: now also U2.8 (Pin_8); no longer U1.8 (Pin_8)
- net LED5: now also U2.9 (Pin_9); no longer U1.9 (Pin_9)
- net LED6: now also U2.10 (Pin_10); no longer U1.10 (Pin_10)
- net LED7: now also U2.11 (Pin_11); no longer U1.11 (Pin_11)
- net LED8: now also U2.12 (Pin_12); no longer U1.12 (Pin_12)
- net LED9: now also U2.13 (Pin_13); no longer U1.13 (Pin_13)
- net SENS_MINUS: now also U1.11 (Pin_11); no longer U2.11 (Pin_11)
- net SENS_PLUS: now also U2.15 (Pin_15); no longer U1.15 (Pin_15)
Changed lines of the file:
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@@
 		(title "Lemon Piano V5.5 Board")
 		(date "2026-07-30")
-		(rev "v0.1.0")
+		(rev "v0.2.0")
 		(company "Lemon Piano")
 		(comment 1 "V5 game board + V5.5 power-entry filter (TVS + Schottky + CLC pi)")
@@
 	(wire
 		(pts
+			(xy 54.61 82.55) (xy 53.34 82.55)
+		)
+		(stroke
+			(width 0)
+			(type default)
+		)
+	)
+	(wire
+		(pts
 			(xy 54.61 90.17) (xy 53.34 90.17)
 		)
@@
 	(wire
 		(pts
-			(xy 54.61 113.03) (xy 53.34 113.03)
-		)
-		(stroke
-			(width 0)
-			(type default)
-		)
-	)
-	(wire
-		(pts
 			(xy 54.61 115.57) (xy 53.34 115.57)
 		)
@@
 	(wire
 		(pts
-			(xy 54.61 118.11) (xy 53.34 118.11)
+			(xy 85.09 90.17) (xy 86.36 90.17)
 		)
 		(stroke
@@
 	(wire
 		(pts
-			(xy 85.09 82.55) (xy 86.36 82.55)
+			(xy 85.09 92.71) (xy 86.36 92.71)
 		)
 		(stroke
@@
 	(wire
 		(pts
-			(xy 85.09 90.17) (xy 86.36 90.17)
+			(xy 85.09 95.25) (xy 86.36 95.25)
 		)
 		(stroke
@@
 	(wire
 		(pts
-			(xy 85.09 92.71) (xy 86.36 92.71)
+			(xy 85.09 97.79) (xy 86.36 97.79)
 		)
 		(stroke
@@
 	(wire
 		(pts
-			(xy 85.09 95.25) (xy 86.36 95.25)
+			(xy 85.09 100.33) (xy 86.36 100.33)
 		)
 		(stroke
@@
 	(wire
 		(pts
-			(xy 85.09 97.79) (xy 86.36 97.79)
+			(xy 85.09 102.87) (xy 86.36 102.87)
 		)
 		(stroke
@@
 	(wire
 		(pts
-			(xy 85.09 100.33) (xy 86.36 100.33)
+			(xy 85.09 105.41) (xy 86.36 105.41)
 		)
 		(stroke
@@
 	(wire
 		(pts
-			(xy 85.09 102.87) (xy 86.36 102.87)
+			(xy 85.09 107.95) (xy 86.36 107.95)
 		)
 		(stroke
@@
 	(wire
 		(pts
-			(xy 85.09 105.41) (xy 86.36 105.41)
+			(xy 85.09 110.49) (xy 86.36 110.49)
 		)
 		(stroke
@@
 	(wire
 		(pts
-			(xy 85.09 107.95) (xy 86.36 107.95)
+			(xy 85.09 113.03) (xy 86.36 113.03)
 		)
 		(stroke
@@
 	(wire
 		(pts
-			(xy 85.09 110.49) (xy 86.36 110.49)
+			(xy 85.09 115.57) (xy 86.36 115.57)
 		)
 		(stroke
@@
 	(wire
 		(pts
-			(xy 85.09 115.57) (xy 86.36 115.57)
+			(xy 85.09 118.11) (xy 86.36 118.11)
 		)
 		(stroke
@@
 		)
 	)
-	(label "GND"
+	(label "BUZZER"
+		(at 53.34 82.55 0)
+		(effects
+			(font
+				(size 1.27 1.27)
+			)
+			(justify left bottom)
+		)
+	)
+	(label "KEY1"
 		(at 53.34 90.17 0)
 		(effects
@@
 		)
 	)
-	(label "LED1"
+	(label "KEY2"
 		(at 53.34 92.71 0)
 		(effects
@@
 		)
 	)
-	(label "LED2"
+	(label "KEY3"
 		(at 53.34 95.25 0)
 		(effects
@@
 		)
 	)
-	(label "LED3"
+	(label "KEY4"
 		(at 53.34 97.79 0)
 		(effects
@@
 		)
 	)
-	(label "LED4"
+	(label "KEY5"
 		(at 53.34 100.33 0)
 		(effects
@@
 		)
 	)
-	(label "LED5"
+	(label "KEY6"
 		(at 53.34 102.87 0)
 		(effects
@@
 		)
 	)
-	(label "LED6"
+	(label "KEY7"
 		(at 53.34 105.41 0)
 		(effects
@@
 		)
 	)
-	(label "LED7"
+	(label "SENS_MINUS"
 		(at 53.34 107.95 0)
 		(effects
@@
 		)
 	)
-	(label "LED8"
+	(label "+5V"
 		(at 53.34 110.49 0)
 		(effects
@@
 		)
 	)
-	(label "LED9"
-		(at 53.34 113.03 0)
-		(effects
-			(font
-				(size 1.27 1.27)
-			)
-			(justify left bottom)
-		)
-	)
-	(label "LED10"
+	(label "GND"
 		(at 53.34 115.57 0)
 		(effects
@@
 		)
 	)
-	(label "SENS_PLUS"
-		(at 53.34 118.11 0)
+	(label "GND"
+		(at 86.36 90.17 0)
 		(effects
 			(font
@@
 		)
 	)
-	(label "BUZZER"
-		(at 86.36 82.55 0)
+	(label "LED1"
+		(at 86.36 92.71 0)
 		(effects
 			(font
@@
 		)
 	)
-	(label "KEY1"
-		(at 86.36 90.17 0)
+	(label "LED2"
+		(at 86.36 95.25 0)
 		(effects
 			(font
@@
 		)
 	)
-	(label "KEY2"
-		(at 86.36 92.71 0)
+	(label "LED3"
+		(at 86.36 97.79 0)
 		(effects
 			(font
@@
 		)
 	)
-	(label "KEY3"
-		(at 86.36 95.25 0)
+	(label "LED4"
+		(at 86.36 100.33 0)
 		(effects
 			(font
@@
 		)
 	)
-	(label "KEY4"
-		(at 86.36 97.79 0)
+	(label "LED5"
+		(at 86.36 102.87 0)
 		(effects
 			(font
@@
 		)
 	)
-	(label "KEY5"
-		(at 86.36 100.33 0)
+	(label "LED6"
+		(at 86.36 105.41 0)
 		(effects
 			(font
@@
 		)
 	)
-	(label "KEY6"
-		(at 86.36 102.87 0)
+	(label "LED7"
+		(at 86.36 107.95 0)
 		(effects
 			(font
@@
 		)
 	)
-	(label "KEY7"
-		(at 86.36 105.41 0)
+	(label "LED8"
+		(at 86.36 110.49 0)
 		(effects
 			(font
@@
 		)
 	)
-	(label "SENS_MINUS"
-		(at 86.36 107.95 0)
+	(label "LED9"
+		(at 86.36 113.03 0)
 		(effects
 			(font
@@
 		)
 	)
-	(label "+5V"
-		(at 86.36 110.49 0)
+	(label "LED10"
+		(at 86.36 115.57 0)
 		(effects
 			(font
@@
 		)
 	)
-	(label "GND"
-		(at 86.36 115.57 0)
+	(label "SENS_PLUS"
+		(at 86.36 118.11 0)
 		(effects
 			(font
@@
 		)
 	)
-	(label "GND"
+	(label "KEY1"
 		(at 115.57 92.71 0)
 		(effects
@@
 		)
 	)
-	(label "KEY7"
+	(label "KEY2"
 		(at 115.57 95.25 0)
 		(effects
@@
 		)
 	)
-	(label "KEY6"
+	(label "KEY3"
 		(at 115.57 97.79 0)
 		(effects
@@
 		)
 	)
-	(label "KEY5"
+	(label "KEY4"
 		(at 115.57 100.33 0)
 		(effects
@@
 		)
 	)
-	(label "KEY4"
+	(label "KEY5"
 		(at 115.57 102.87 0)
 		(effects
@@
 		)
 	)
-	(label "KEY3"
+	(label "KEY6"
 		(at 115.57 105.41 0)
 		(effects
@@
 		)
 	)
-	(label "KEY2"
+	(label "KEY7"
 		(at 115.57 107.95 0)
 		(effects
@@
 		)
 	)
-	(label "KEY1"
+	(label "GND"
 		(at 115.57 110.49 0)
 		(effects
@@
 	)
 	(no_connect
-		(at 54.61 82.55)
-	)
-	(no_connect
 		(at 54.61 85.09)
 	)
@@
 	)
 	(no_connect
-		(at 85.09 85.09)
+		(at 54.61 113.03)
 	)
 	(no_connect
-		(at 85.09 87.63)
+		(at 54.61 118.11)
 	)
 	(no_connect
-		(at 85.09 113.03)
+		(at 85.09 82.55)
 	)
 	(no_connect
-		(at 85.09 118.11)
+		(at 85.09 85.09)
+	)
+	(no_connect
+		(at 85.09 87.63)
 	)
 	(sheet_instances

Commit message: feat(pcb): v0.4.0 — 120x40 remake, centred Nano, external-button headers
Complete floor-plan remake to the user's distribution spec. The V5.5
circuit is unchanged (no value, pin or part invented); only the board
frame and its interface changed.

- 120 x 40 mm frame (was 100 x 30), KiCad frame x 90..210 / y 100..140.
  Anchor dividers at x=100/200; four M2 holes to the corners at 5 mm
  insets (95/205 x 105/135), mirror-symmetric about x=150 and y=120.
- Nano socket centred on the board (pin field x 132.22..167.78, rows
  y 112.38/127.62), mini-USB still WEST. Centring it turned the USB
  corridor from a 14 mm sliver into a 42 mm strip, so the corridor is
  redefined as the band a cable needs (x < 130.4, y 113..127) and kept
  completely part-free, checked against real courtyard boxes.
- Whole 5 V filter in the west block, folded around that corridor: VIN
  section on the south strip (J1 -> D1 -> D2), VRAW/+5V on the north
  strip (C1 -> L1), output reservoir C3 at the south-strip east end.
  Three 8 mm radial parts do not fit one 27 mm strip, which forced the
  split. D2 at rot=180 so the chain reads west->east with no doubling
  back; EXPECTED_PADS locks that new rotation convention.
- 5 V entry is now a 2-pin 2.54 mm header (J1), replacing the Phoenix
  screw terminal, per the user's "2 pines". Same nets and polarity.
- A parallel 2-pin header per SENS button (J3 || SW1 on /SENS_PLUS,
  J4 || SW2 on /SENS_MINUS), each directly east of its button, so an
  external panel button plugs in without cutting a trace.
- Keys header centred on the south edge (pin centre exactly x=150);
  SENS button pair centred on y=120; LED bar centred over its D2..D11
  pin span so the fan legs stay short at both ends.
- Buzzer to the NE corner — the only place its 12.56 mm courtyard fits
  once the button column and EXT headers claim their x-lanes. Costs a
  ~58 mm /BUZZER run (piezo square wave over a solid plane: harmless).
- Title block moved into the USB corridor; KEYS word moved ea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
Parts:
- added J3: SENS+_EXT, Connector_PinHeader_2.54mm:PinHeader_1x02_P2.54mm_Vertical, symbol Connector_Generic:Conn_01x02
- added J4: SENS-_EXT, Connector_PinHeader_2.54mm:PinHeader_1x02_P2.54mm_Vertical, symbol Connector_Generic:Conn_01x02
- J1: footprint TerminalBlock_Phoenix:TerminalBlock_Phoenix_MKDS-1,5-2-5.08_1x02_P5.08mm_Horizontal -> Connector_PinHeader_2.54mm:PinHeader_1x02_P2.54mm_Vertical; symbol Connector:Screw_Terminal_01x02 -> Connector_Generic:Conn_01x02
Connections:
- net GND: now also J3.2 (Pin_2), J4.2 (Pin_2)
- net SENS_MINUS: now also J4.1 (Pin_1)
- net SENS_PLUS: now also J3.1 (Pin_1)
Changed lines of the file:
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@@
 		(title "Lemon Piano V5.5 Board")
 		(date "2026-07-30")
-		(rev "v0.3.0")
+		(rev "v0.4.0")
 		(company "Lemon Piano")
 		(comment 1 "V5 game board + V5.5 power-entry filter (TVS + Schottky + CLC pi)")
@@
 	)
 	(symbol
-		(lib_id "Connector:Screw_Terminal_01x02")
+		(lib_id "Connector_Generic:Conn_01x02")
 		(at 30.48 39.37 0)
 		(unit 1)
@@
 			)
 		)
-		(property "Footprint" "TerminalBlock_Phoenix:TerminalBlock_Phoenix_MKDS-1,5-2-5.08_1x02_P5.08mm_Horizontal"
+		(property "Footprint" "Connector_PinHeader_2.54mm:PinHeader_1x02_P2.54mm_Vertical"
 			(at 30.48 39.37 0.0000)
 			(effects
@@
 	)
 	(symbol
+		(lib_id "Connector_Generic:Conn_01x02")
+		(at 30.48 124.46 0)
+		(unit 1)
+		(exclude_from_sim no)
+		(in_bom yes)
+		(on_board yes)
+		(dnp no)
+		(fields_autoplaced no)
+		(property "Reference" "J3"
+			(at 30.48 127 0.0000)
+			(effects
+				(font
+					(size 1.27 1.27)
+				)
+				(justify left)
+			)
+		)
+		(property "Value" "SENS+_EXT"
+			(at 30.48 119.38 0.0000)
+			(effects
+				(font
+					(size 1.27 1.27)
+				)
+				(justify left)
+			)
+		)
+		(property "Footprint" "Connector_PinHeader_2.54mm:PinHeader_1x02_P2.54mm_Vertical"
+			(at 30.48 124.46 0.0000)
+			(effects
+				(font
+					(size 1.27 1.27)
+				)
+				(hide yes)
+			)
+		)
+		(pin "1"
+		)
+		(pin "2"
+		)
+		(instances
+			(project "lemon-piano"
+				(path "/c97fa168-2ffe-53ab-a801-ca02fb3766e2"
+					(reference "J3")
+					(unit 1)
+				)
+			)
+		)
+	)
+	(symbol
+		(lib_id "Connector_Generic:Conn_01x02")
+		(at 30.48 139.7 0)
+		(unit 1)
+		(exclude_from_sim no)
+		(in_bom yes)
+		(on_board yes)
+		(dnp no)
+		(fields_autoplaced no)
+		(property "Reference" "J4"
+			(at 30.48 142.24 0.0000)
+			(effects
+				(font
+					(size 1.27 1.27)
+				)
+				(justify left)
+			)
+		)
+		(property "Value" "SENS-_EXT"
+			(at 30.48 134.62 0.0000)
+			(effects
+				(font
+					(size 1.27 1.27)
+				)
+				(justify left)
+			)
+		)
+		(property "Footprint" "Connector_PinHeader_2.54mm:PinHeader_1x02_P2.54mm_Vertical"
+			(at 30.48 139.7 0.0000)
+			(effects
+				(font
+					(size 1.27 1.27)
+				)
+				(hide yes)
+			)
+		)
+		(pin "1"
+		)
+		(pin "2"
+		)
+		(instances
+			(project "lemon-piano"
+				(path "/c97fa168-2ffe-53ab-a801-ca02fb3766e2"
+					(reference "J4")
+					(unit 1)
+				)
+			)
+		)
+	)
+	(symbol
 		(lib_id "power:PWR_FLAG")
 		(at 30.48 25.4 0)
@@
 	(wire
 		(pts
+			(xy 25.4 124.46) (xy 24.13 124.46)
+		)
+		(stroke
+			(width 0)
+			(type default)
+		)
+	)
+	(wire
+		(pts
+			(xy 25.4 127) (xy 24.13 127)
+		)
+		(stroke
+			(width 0)
+			(type default)
+		)
+	)
+	(wire
+		(pts
+			(xy 25.4 139.7) (xy 24.13 139.7)
+		)
+		(stroke
+			(width 0)
+			(type default)
+		)
+	)
+	(wire
+		(pts
+			(xy 25.4 142.24) (xy 24.13 142.24)
+		)
+		(stroke
+			(width 0)
+			(type default)
+		)
+	)
+	(wire
+		(pts
 			(xy 30.48 25.4) (xy 30.48 26.67)
 		)
@@
 		(effects
 			(font
+				(size 1.27 1.27)
+			)
+			(justify left bottom)
+		)
+	)
+	(label "SENS_PLUS"
+		(at 24.13 124.46 0)
+		(effects
+			(font
+				(size 1.27 1.27)
+			)
+			(justify left bottom)
+		)
+	)
+	(label "GND"
+		(at 24.13 127 0)
+		(effects
+			(font
+				(size 1.27 1.27)
+			)
+			(justify left bottom)
+		)
+	)
+	(label "SENS_MINUS"
+		(at 24.13 139.7 0)
+		(effects
+			(font
+				(size 1.27 1.27)
+			)
+			(justify left bottom)
+		)
+	)
+	(label "GND"
+		(at 24.13 142.24 0)
+		(effects
+			(font

Commit message: feat(pcb): v0.6.0 — J5, 2-pin aux speaker output in parallel with the buzzer
User request: two pins for an external speaker.

- New 2-pin header J5 (silk "SPK") on the SAME two nodes as the buzzer:
  pad 1 on /BUZZER (the D13 drive line), pad 2 on /GND. Placed immediately
  west of BUZ1 with a 5.18 mm courtyard gap, same pattern as the SENS
  external-button headers (ADR-026). Nothing is switched or cut - the
  on-board buzzer keeps sounding and whatever is plugged into J5 sees
  exactly the same signal.

- LOAD LIMIT, documented in ADR-034 and the README assembly notes. The
  buzzer is a PASSIVE piezo driven straight off the pin ("no series
  resistor needed", versions/v0-buzzer/HARDWARE.md), i.e. a high-impedance
  load of a few mA. A bare 4-8 ohm dynamic voice coil is not: at 5 V it
  would ask for roughly 600 mA against the ATmega328P's 40 mA absolute
  maximum (20 mA recommended) per pin, and would damage D13. J5 is
  therefore rated for another piezo element or an AMPLIFIED speaker module
  (PAM8403 / LM386 / powered PC speakers - all high-impedance inputs); a
  raw speaker only through an amplifier.

  No series resistor or amplifier was added to the board: the sources
  define a directly-driven passive buzzer, and inventing parts or values no
  source specifies is against the project's rules. A driver stage is a
  versions/ circuit change first, not a PCB-layer improvisation.

- geometry_gate gains a check that J5 stays adjacent to the buzzer it
  parallels (28 checks now). verify_placement covers 74 pad-net-function
  pairs (was 73). Schematic is 48 symbols (was 47).

- Fixed a pre-existing documentation error found while editing NETLIST.md:
  the U1/U2 rows in the component table had their descriptions swapped. U1
  is the ANALOG column (D13,3V3,AREF,A0..A7,5V,RST,GND,VIN), U2 the DIGITAL
  one (TX1,RX0,RST,GND,D2..D12). The pad-net tables and the ground truth
  were always right; only that table's prose was wrong.

Verification on the committed board: DRC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
Parts:
- added J4: SENS-_EXT, Connector_PinHeader_2.54mm:PinHeader_1x02_P2.54mm_Vertical, symbol Connector_Generic:Conn_01x02
- J3: renamed from J4; value SENS-_EXT -> SENS+_EXT
- J5: renamed from SW1; value SENS+ -> SPK_OUT; footprint Button_Switch_THT:SW_PUSH_6mm -> Connector_PinHeader_2.54mm:PinHeader_1x02_P2.54mm_Vertical; symbol Switch:SW_Push -> Connector_Generic:Conn_01x02
- SW1: renamed from SW2; value SENS- -> SENS+
- SW2: renamed from J3; value SENS+_EXT -> SENS-; footprint Connector_PinHeader_2.54mm:PinHeader_1x02_P2.54mm_Vertical -> Button_Switch_THT:SW_PUSH_6mm; symbol Connector_Generic:Conn_01x02 -> Switch:SW_Push
Connections:
- net BUZZER: now also J5.1 (Pin_1)
- net GND: now also J4.2 (Pin_2)
- net SENS_MINUS: now also SW2.1, J4.1 (Pin_1); no longer J3.1 (Pin_1), SW1.1
- net SENS_PLUS: now also J3.1 (Pin_1), SW1.1; no longer J5.1, SW2.1 (Pin_1)
Other:
- moved on the sheet: J3, SW1
Changed lines of the file:
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@@
 		(title "Lemon Piano V5.5 Board")
 		(date "2026-07-30")
-		(rev "v0.5.1")
+		(rev "v0.6.0")
 		(company "Lemon Piano")
 		(comment 1 "V5 game board + V5.5 power-entry filter (TVS + Schottky + CLC pi)")
@@
 	)
 	(symbol
+		(lib_id "Connector_Generic:Conn_01x02")
+		(at 15.24 80.01 0)
+		(unit 1)
+		(exclude_from_sim no)
+		(in_bom yes)
+		(on_board yes)
+		(dnp no)
+		(fields_autoplaced no)
+		(property "Reference" "J5"
+			(at 15.24 82.55 0.0000)
+			(effects
+				(font
+					(size 1.27 1.27)
+				)
+				(justify left)
+			)
+		)
+		(property "Value" "SPK_OUT"
+			(at 15.24 74.93 0.0000)
+			(effects
+				(font
+					(size 1.27 1.27)
+				)
+				(justify left)
+			)
+		)
+		(property "Footprint" "Connector_PinHeader_2.54mm:PinHeader_1x02_P2.54mm_Vertical"
+			(at 15.24 80.01 0.0000)
+			(effects
+				(font
+					(size 1.27 1.27)
+				)
+				(hide yes)
+			)
+		)
+		(pin "1"
+		)
+		(pin "2"
+		)
+		(instances
+			(project "lemon-piano"
+				(path "/c97fa168-2ffe-53ab-a801-ca02fb3766e2"
+					(reference "J5")
+					(unit 1)
+				)
+			)
+		)
+	)
+	(symbol
 		(lib_id "Switch:SW_Push")
 		(at 30.48 95.25 0)
@@
 	(wire
 		(pts
+			(xy 10.16 80.01) (xy 8.89 80.01)
+		)
+		(stroke
+			(width 0)
+			(type default)
+		)
+	)
+	(wire
+		(pts
+			(xy 10.16 82.55) (xy 8.89 82.55)
+		)
+		(stroke
+			(width 0)
+			(type default)
+		)
+	)
+	(wire
+		(pts
 			(xy 25.4 95.25) (xy 24.13 95.25)
 		)
@@
 		(effects
 			(font
+				(size 1.27 1.27)
+			)
+			(justify left bottom)
+		)
+	)
+	(label "BUZZER"
+		(at 8.89 80.01 0)
+		(effects
+			(font
+				(size 1.27 1.27)
+			)
+			(justify left bottom)
+		)
+	)
+	(label "GND"
+		(at 8.89 82.55 0)
+		(effects
+			(font
